File: pcb/Wattuino-Uno_v10.brd (EAGLE design)
At the start: 68.6 x 53.3 mm, 61 parts, among them IC1 ATMEGA328-PU, IC2 FT231XQ, IC3 LDO-TS1117CW-5V, IC4 LDO-TS9011-3V3, J2 USB-B-H, J3 USB-MICRO, Q1 16MHz, X1 PASSER-07, X2 PASSER-07, X3 PASSER-07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

Commit message: updated schematics
Parts:
- R10: value 100k -> 10k
- R12: value 1k -> 10k
Changed lines of the file:
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@@
 <attribute name="VALUE" x="17.78" y="23.01875" size="0.8128" layer="27" font="vector" ratio="10" align="center"/>
 </element>
-<element name="R10" library="we-rcl" package="C0402" value="100k" x="10.16" y="28.8925" smashed="yes">
+<element name="R10" library="we-rcl" package="C0402" value="10k" x="10.16" y="28.8925" smashed="yes">
 <attribute name="NAME" x="10.16" y="26.82875" size="0.8128" layer="25" font="vector" ratio="10" rot="R90" align="center"/>
 <attribute name="VALUE" x="10.4775" y="30.48" size="0.8128" layer="27" font="vector" ratio="10" rot="R180" align="center"/>
@@
 <attribute name="VALUE" x="15.875" y="11.43" size="0.8128" layer="27" font="vector" align="center"/>
 </element>
-<element name="R12" library="we-rcl" package="C0402" value="1k" x="8.5725" y="28.8925" smashed="yes" rot="R180">
+<element name="R12" library="we-rcl" package="C0402" value="10k" x="8.5725" y="28.8925" smashed="yes" rot="R180">
 <attribute name="NAME" x="8.5725" y="26.82875" size="0.8128" layer="25" font="vector" ratio="10" rot="R90" align="center"/>
 <attribute name="VALUE" x="8.255" y="30.48" size="0.8128" layer="27" font="vector" ratio="10" rot="R180" align="center"/>
