File: pcb/Wattuino-Uno_v10.sch (EAGLE design)
At the start: 61 parts, among them IC1 ATMEGA328-PU, IC2 FT231XQ, IC3 LDO-TS1117CW-5V, IC4 LDO-TS9011-3V3, J2 USB-B-H, J3 USB-MICRO, Q1 16MHz, X1 PASSER-07, X2 PASSER-07, X3 PASSER-07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

Commit message: updated schematics
Parts:
- R10: value 100k -> 10k
- R12: value 1k -> 10k
Changed lines of the file:
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@@
 <setting verticaltext="up"/>
 </settings>
-<grid distance="0.05" unitdist="inch" unit="inch" style="lines" multiple="1" display="yes" altdistance="0.01" altunitdist="inch" altunit="inch"/>
+<grid distance="0.05" unitdist="inch" unit="inch" style="lines" multiple="1" display="yes" altdistance="0.025" altunitdist="inch" altunit="inch"/>
 <layers>
 <layer number="1" name="Top" color="4" fill="1" visible="no" active="no"/>
@@
 <part name="P+4" library="supply1" deviceset="+5V" device=""/>
 <part name="C12" library="we-rcl" deviceset="CAPACITOR" device="-0402" value="100n"/>
-<part name="R10" library="we-rcl" deviceset="RESISTOR" device="-0402" value="100k"/>
+<part name="R10" library="we-rcl" deviceset="RESISTOR" device="-0402" value="10k"/>
 <part name="F1" library="we-rcl" deviceset="FUSE" device="-0805" value="500mA"/>
 <part name="RX" library="we-opto" deviceset="LED" device="-0603" value="red"/>
@@
 <part name="+3V6" library="supply1" deviceset="+3V3" device=""/>
 <part name="D2" library="we-rcl" deviceset="D_SCHOTTKY" device="-SS14"/>
-<part name="R12" library="we-rcl" deviceset="RESISTOR" device="-0402" value="1k"/>
+<part name="R12" library="we-rcl" deviceset="RESISTOR" device="-0402" value="10k"/>
 </parts>
 <sheets>
