File: hardware/Wattuino-Nanite85_v10.brd (EAGLE design)
At the start: 17.5 x 10.2 mm, 18 parts, among them IC2 ATTINY85-MU, J1 USB-MICRO, J2 MA04-1, J3 MA04-1, SW1 SW-TACTILE-PTS840P, X1 PASSER-07, X2 PASSER-07, X3 PASSER-07

Commit message: updated layout and schematics
Changed lines of the file:
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@@
 <?xml version="1.0" encoding="utf-8"?>
 <!DOCTYPE eagle SYSTEM "eagle.dtd">
-<eagle version="7.2.0">
+<eagle version="7.5.0">
 <drawing>
 <settings>
@@
 <wire x1="6.17375" y1="3.76" x2="6.19125" y2="3.7775" width="0.2032" layer="1"/>
 <wire x1="1.49625" y1="4.1175" x2="1.49625" y2="6.0425" width="0.3048" layer="1"/>
-<wire x1="6.3246" y1="7.3875" x2="6.3246" y2="6.80085" width="0.3048" layer="1"/>
+<wire x1="6.3246" y1="7.4375" x2="6.3246" y2="6.80085" width="0.3048" layer="1"/>
 <wire x1="6.3246" y1="6.80085" x2="6.19125" y2="6.6675" width="0.3048" layer="1"/>
 <wire x1="6.19125" y1="6.6675" x2="6.19125" y2="6.3825" width="0.3048" layer="1"/>
@@
 <via x="14.12875" y="6.985" extent="1-16" drill="0.3"/>
 <contactref element="IC2" pad="TP"/>
-<wire x1="6.3246" y1="7.3875" x2="6.2396" y2="7.3025" width="0.2032" layer="1"/>
+<wire x1="6.3246" y1="7.4375" x2="6.2396" y2="7.3025" width="0.2032" layer="1"/>
 <wire x1="6.2396" y1="7.3025" x2="6.19125" y2="7.3025" width="0.2032" layer="1"/>
 </signal>
@@
 <contactref element="R4" pad="1"/>
 <contactref element="J3" pad="1"/>
-<wire x1="6.3246" y1="8.4875" x2="6.365" y2="8.5875" width="0.3048" layer="1"/>
+<wire x1="6.3246" y1="8.4375" x2="6.365" y2="8.5875" width="0.3048" layer="1"/>
 <wire x1="8.08125" y1="8.905" x2="8.09625" y2="8.89" width="0.2032" layer="1"/>
 <wire x1="10.90625" y1="6.98" x2="10.90625" y2="7.35" width="0.3048" layer="1"/>
@@
 <wire x1="6.3246" y1="1.11125" x2="6.35" y2="1.11125" width="0.3048" layer="16"/>
 <wire x1="6.35" y1="1.11125" x2="6.50875" y2="1.27" width="0.3048" layer="16"/>
-<wire x1="6.3246" y1="1.6725" x2="6.3246" y2="1.11125" width="0.3048" layer="1"/>
-<wire x1="8.6653" y1="6.50875" x2="8.6653" y2="7.62" width="0.3048" layer="1"/>
+<wire x1="6.3246" y1="1.7225" x2="6.3246" y2="1.11125" width="0.3048" layer="1"/>
+<wire x1="8.6153" y1="6.50875" x2="8.6653" y2="7.62" width="0.3048" layer="1"/>
 <wire x1="8.6653" y1="7.62" x2="8.6653" y2="8.32095" width="0.3048" layer="1"/>
 <wire x1="10.63625" y1="7.62" x2="8.6653" y2="7.62" width="0.3048" layer="1"/>
@@
 <wire x1="8.89" y1="2.54" x2="8.89" y2="5.3467" width="0.2032" layer="16"/>
 <wire x1="8.89" y1="5.3467" x2="8.9408" y2="5.3975" width="0.2032" layer="16"/>
-<wire x1="8.6653" y1="4.60375" x2="8.6653" y2="5.122" width="0.2032" layer="1"/>
+<wire x1="8.6153" y1="4.60375" x2="8.6653" y2="5.122" width="0.2032" layer="1"/>
 <wire x1="8.6653" y1="5.122" x2="8.9408" y2="5.3975" width="0.2032" layer="1"/>
 </signal>
@@
 <wire x1="6.14375" y1="5.73" x2="6.19125" y2="5.6825" width="0.2032" layer="1"/>
 <wire x1="6.19125" y1="5.6825" x2="7.5653" y2="5.6825" width="0.2032" layer="1"/>
-<wire x1="7.5653" y1="5.6825" x2="7.5653" y2="4.60375" width="0.2032" layer="1"/>
-<wire x1="7.5653" y1="6.50875" x2="7.5653" y2="5.6825" width="0.2032" layer="1"/>
+<wire x1="7.5653" y1="5.6825" x2="7.6153" y2="4.60375" width="0.2032" layer="1"/>
+<wire x1="7.6153" y1="6.50875" x2="7.5653" y2="5.6825" width="0.2032" layer="1"/>
 </signal>
 <signal name="PB4">
@@
 <wire x1="9.68375" y1="3.175" x2="11.27125" y2="3.175" width="0.2032" layer="16"/>
 <wire x1="11.27125" y1="3.175" x2="13.17625" y2="1.27" width="0.2032" layer="16"/>
-<wire x1="8.6653" y1="3.33375" x2="9.525" y2="3.33375" width="0.2032" layer="1"/>
+<wire x1="8.6153" y1="3.33375" x2="9.525" y2="3.33375" width="0.2032" layer="1"/>
 <wire x1="9.525" y1="3.33375" x2="9.68375" y2="3.175" width="0.2032" layer="1"/>
 </signal>
@@
 <contactref element="J1" pad="D+"/>
 <contactref element="D1" pad="C"/>
-<wire x1="7.5653" y1="3.33375" x2="7.1628" y2="3.33375" width="0.2032" layer="1"/>
+<wire x1="7.6153" y1="3.33375" x2="7.1628" y2="3.33375" width="0.2032" layer="1"/>
 <wire x1="7.1628" y1="3.33375" x2="6.82625" y2="3.81" width="0.2032" layer="1" curve="-90"/>
 <wire x1="6.82625" y1="3.81" x2="6.82625" y2="3.96875" width="0.2032" layer="1"/>
@@
 <wire x1="10.90625" y1="3.18" x2="10.8" y2="3.18" width="0.3048" layer="1"/>
 <wire x1="10.8" y1="3.18" x2="10.00125" y2="2.38125" width="0.3048" layer="1"/>
-<wire x1="6.3246" y1="2.7725" x2="6.49375" y2="2.8725" width="0.2032" layer="1"/>
+<wire x1="6.3246" y1="2.7225" x2="6.49375" y2="2.8725" width="0.2032" layer="1"/>
 <wire x1="6.49375" y1="2.8725" x2="8.09625" y2="1.27" width="0.2032" layer="1"/>
 <wire x1="7.82955" y1="5.87375" x2="7.82955" y2="1.5367" width="0.3048" layer="16"/>
