File: hardware/Wattuino-Nanite85_v10.sch (EAGLE design)
At the start: 18 parts, among them IC2 ATTINY85-MU, J1 USB-MICRO, J2 MA04-1, J3 MA04-1, SW1 SW-TACTILE-PTS840P, X1 PASSER-07, X2 PASSER-07, X3 PASSER-07

Commit message: updated layout and schematics
Connections:
- net PB3: now also IC2.(XTAL1/CLKI/ADC3/!OC1B!)PB3; no longer IC2.(XTAL1/ADC3/!OC1B!)PB3
- net PB4: now also IC2.(XTAL2/CLKO/ADC2/OC1B)PB4; no longer IC2.(XTAL2/ADC2/OC1B)PB4
Changed lines of the file:
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@@
 <?xml version="1.0" encoding="utf-8"?>
 <!DOCTYPE eagle SYSTEM "eagle.dtd">
-<eagle version="7.3.0">
+<eagle version="7.5.0">
 <drawing>
 <settings>
@@
 <net name="PB3" class="0">
 <segment>
-<pinref part="IC2" gate="IC" pin="(XTAL1/ADC3/!OC1B!)PB3"/>
+<pinref part="IC2" gate="IC" pin="(XTAL1/CLKI/ADC3/!OC1B!)PB3"/>
 <pinref part="R2" gate="R" pin="1"/>
 <wire x1="106.68" y1="118.11" x2="116.84" y2="118.11" width="0.1524" layer="91"/>
@@
 <net name="PB4" class="0">
 <segment>
-<pinref part="IC2" gate="IC" pin="(XTAL2/ADC2/OC1B)PB4"/>
+<pinref part="IC2" gate="IC" pin="(XTAL2/CLKO/ADC2/OC1B)PB4"/>
 <wire x1="106.68" y1="115.57" x2="116.84" y2="115.57" width="0.1524" layer="91"/>
 <wire x1="116.84" y1="115.57" x2="119.38" y2="118.11" width="0.1524" layer="91"/>
