File: hardware/Wattuino-Uno_v10.brd (EAGLE design)
At the start: 68.6 x 53.3 mm, 61 parts, among them IC1 ATMEGA328-PU, IC2 FT231XQ, IC3 LDO-TS1117CW-5V, IC4 LDO-TS9011-3V3, J2 USB-B-H, J3 USB-MICRO, Q1 16MHz, X1 PASSER-07, X2 PASSER-07, X3 PASSER-07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

Commit message: updated schematics
Parts:
- L1: value (none) -> 10u
Changed lines of the file:
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@@
 <attribute name="VALUE" x="23.1775" y="5.3975" size="0.8128" layer="27" font="vector" ratio="10" rot="R180" align="center"/>
 </element>
-<element name="L1" library="we-rcl" package="C0603" value="" x="40.005" y="9.525" smashed="yes" rot="R90">
+<element name="L1" library="we-rcl" package="C0603" value="10u" x="40.005" y="9.525" smashed="yes" rot="R90">
 <attribute name="NAME" x="40.005" y="10.795" size="0.8128" layer="25" font="vector" ratio="10" align="center"/>
 <attribute name="VALUE" x="40.005" y="10.795" size="0.8128" layer="27" font="vector" ratio="10" align="center"/>
