File: hardware/Wattuino-Nanite841_v10.brd (EAGLE design)
At the start: 24.1 x 10.2 mm, 20 parts, among them IC1 ATTINY841-MU, J1 USB-MICRO, J2 MA07-1, J3 MA07-1, SW1 SW-TACTILE-PTS840P, X1 PASSER-07, X2 PASSER-07, X3 PASSER-07

Commit message: updated layout and schematics
Changed lines of the file:
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@@
 <?xml version="1.0" encoding="utf-8"?>
 <!DOCTYPE eagle SYSTEM "eagle.dtd">
-<eagle version="7.3.0">
+<eagle version="7.5.0">
 <drawing>
 <settings>
@@
 <contactref element="J3" pad="1"/>
 <wire x1="13.18125" y1="5.08" x2="15.08125" y2="5.08" width="0.2032" layer="1"/>
-<wire x1="11.7729" y1="5.63" x2="12.05475" y2="5.63" width="0.3048" layer="1"/>
+<wire x1="11.7729" y1="5.58" x2="12.05475" y2="5.63" width="0.3048" layer="1"/>
 <wire x1="12.05475" y1="5.63" x2="12.60475" y2="5.08" width="0.3048" layer="1"/>
 <wire x1="13.18125" y1="5.08" x2="12.60475" y2="5.08" width="0.3048" layer="1"/>
@@
 <contactref element="R5" pad="2"/>
 <via x="8.73125" y="5.7785" extent="1-16" drill="0.3" diameter="0.254"/>
-<wire x1="11.7729" y1="4.53" x2="10.5205" y2="4.53" width="0.3048" layer="1"/>
-<wire x1="10.5205" y1="4.53" x2="10.414" y2="4.4235" width="0.3048" layer="1"/>
-<wire x1="10.414" y1="5.7365" x2="10.414" y2="4.6365" width="0.3048" layer="1"/>
+<wire x1="11.7729" y1="4.58" x2="10.5205" y2="4.53" width="0.3048" layer="1"/>
+<wire x1="10.5205" y1="4.53" x2="10.414" y2="4.3735" width="0.3048" layer="1"/>
+<wire x1="10.414" y1="5.7865" x2="10.414" y2="4.6365" width="0.3048" layer="1"/>
 <wire x1="10.414" y1="4.6365" x2="10.5205" y2="4.53" width="0.3048" layer="1"/>
 <wire x1="7.3025" y1="1.27" x2="7.3025" y2="5.08" width="0.3048" layer="16"/>
@@
 <wire x1="8.001" y1="5.7785" x2="7.3025" y2="5.08" width="0.3048" layer="16"/>
 <wire x1="8.73125" y1="5.7785" x2="10.372" y2="5.7785" width="0.3048" layer="1"/>
-<wire x1="10.372" y1="5.7785" x2="10.414" y2="5.7365" width="0.3048" layer="1"/>
+<wire x1="10.372" y1="5.7785" x2="10.414" y2="5.7865" width="0.3048" layer="1"/>
 <wire x1="8.73125" y1="5.7785" x2="8.73125" y2="6.80475" width="0.3048" layer="1"/>
-<wire x1="8.73125" y1="6.80475" x2="8.70975" y2="6.82625" width="0.3048" layer="1"/>
+<wire x1="8.73125" y1="6.80475" x2="8.65975" y2="6.82625" width="0.3048" layer="1"/>
 <wire x1="13.18125" y1="4.58" x2="11.8229" y2="4.58" width="0.3048" layer="1"/>
-<wire x1="11.8229" y1="4.58" x2="11.7729" y2="4.53" width="0.3048" layer="1"/>
+<wire x1="11.8229" y1="4.58" x2="11.7729" y2="4.58" width="0.3048" layer="1"/>
 <wire x1="7.3025" y1="1.27" x2="7.366" y2="1.27" width="0.254" layer="16"/>
 </signal>
@@
 <contactref element="J2" pad="6"/>
 <contactref element="R3" pad="1"/>
-<wire x1="8.70975" y1="3.33375" x2="8.70975" y2="2.46625" width="0.2032" layer="1"/>
+<wire x1="8.65975" y1="3.33375" x2="8.70975" y2="2.46625" width="0.2032" layer="1"/>
 <wire x1="8.70975" y1="2.46625" x2="9.906" y2="1.27" width="0.2032" layer="1"/>
 <wire x1="14.08125" y1="3.18" x2="12.99075" y2="3.18" width="0.2032" layer="1"/>
@@
 <wire x1="6.14375" y1="5.73" x2="6.19125" y2="5.6825" width="0.2032" layer="1"/>
 <wire x1="6.19125" y1="5.6825" x2="7.60975" y2="5.6825" width="0.2032" layer="1"/>
-<wire x1="7.60975" y1="5.6825" x2="7.60975" y2="4.60375" width="0.2032" layer="1"/>
-<wire x1="7.60975" y1="6.82625" x2="7.60975" y2="5.6825" width="0.2032" layer="1"/>
+<wire x1="7.60975" y1="5.6825" x2="7.65975" y2="4.60375" width="0.2032" layer="1"/>
+<wire x1="7.65975" y1="6.82625" x2="7.60975" y2="5.6825" width="0.2032" layer="1"/>
 </signal>
 <signal name="PB1">
@@
 <contactref element="IC1" pad="12"/>
 <via x="9.2075" y="4.60375" extent="1-16" drill="0.3" diameter="0.254"/>
-<wire x1="8.70975" y1="4.60375" x2="9.2075" y2="4.60375" width="0.2032" layer="1"/>
+<wire x1="8.65975" y1="4.60375" x2="9.2075" y2="4.60375" width="0.2032" layer="1"/>
 <wire x1="14.58125" y1="3.18" x2="14.58125" y2="2.675" width="0.254" layer="1"/>
 <wire x1="14.58125" y1="2.675" x2="14.31925" y2="2.413" width="0.254" layer="1"/>
@@
 <wire x1="6.82625" y1="4.09575" x2="6.82625" y2="3.90525" width="0.2032" layer="1"/>
 <wire x1="6.82625" y1="3.90525" x2="7.39775" y2="3.33375" width="0.2032" layer="1" curve="90"/>
-<wire x1="7.39775" y1="3.33375" x2="7.60975" y2="3.33375" width="0.2032" layer="1"/>
+<wire x1="7.39775" y1="3.33375" x2="7.65975" y2="3.33375" width="0.2032" layer="1"/>
 <wire x1="6.19125" y1="4.4775" x2="6.381" y2="4.4775" width="0.2032" layer="1"/>
 <wire x1="6.381" y1="4.4775" x2="6.38175" y2="4.47675" width="0.2032" layer="1" curve="-90"/>
@@
 <via x="20.955" y="5.08" extent="1-16" drill="0.3" diameter="0.254"/>
 <via x="11.7475" y="3.429" extent="1-16" drill="0.3" diameter="0.254"/>
-<wire x1="10.414" y1="3.3235" x2="11.642" y2="3.3235" width="0.254" layer="1"/>
+<wire x1="10.414" y1="3.3735" x2="11.642" y2="3.3235" width="0.254" layer="1"/>
 <wire x1="11.642" y1="3.3235" x2="11.7475" y2="3.429" width="0.254" layer="1"/>
 <wire x1="21.9195" y1="5.08" x2="21.9195" y2="3.18" width="0.254" layer="1"/>
@@
 <via x="19.52625" y="6.604" extent="1-16" drill="0.3" diameter="0.254"/>
 <via x="11.7475" y="6.731" extent="1-16" drill="0.3" diameter="0.254"/>
-<wire x1="10.414" y1="6.8365" x2="11.642" y2="6.8365" width="0.254" layer="1"/>
+<wire x1="10.414" y1="6.7865" x2="11.642" y2="6.8365" width="0.254" layer="1"/>
 <wire x1="11.642" y1="6.8365" x2="11.7475" y2="6.731" width="0.254" layer="1"/>
 <wire x1="19.52625" y1="5.83" x2="19.52625" y2="6.604" width="0.2032" layer="1"/>
