File: hardware/Wattuino-RC_v10.sch (EAGLE design)
At the start: 144 parts, among them IC1 ATSAMW25-MR510PB, IC2 74LVC244PW, IC3 A3909-LY, IC4 A3909-LY, IC5 VREG-TS1117CW-3V3, IC6 AP65200-SP, J1 JST3-B3B-PH-K, J2 JST3-B3B-PH-K, J3 JST3-B3B-PH-K, J4 JST3-B3B-PH-K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

Commit message: updated schematics
Parts:
- D1, D2, D5, D6: value 2A/16V -> 2A/20V
Other:
- note added: "1x MosFet"
- note added: "1x Power Switch"
- note added: "1x SPI"
- note added: "1x UART"
- note added: "2x A3909"
- note added: "2x I2C"
- note added: "4x Full Bridges"
- note added: "5V tolerant"
- note added: "7-14V Ext. Power or 5V USB"
- note added: "7x IOs"
- note added: "ARM Cortex-M0+ with USB + WiFi/WLAN"
- note added: "Motor Driver"
- note added: "Power Supply"
- note added: "SAMD21 + WINC1500"
- note added: "SAMW25 Module"
- note added: "up to 1A/phase"
- note added: "up to 2A"
Changed lines of the file:
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@@
 <setting verticaltext="up"/>
 </settings>
-<grid distance="0.1" unitdist="inch" unit="inch" style="lines" multiple="1" display="no" altdistance="0.01" altunitdist="inch" altunit="inch"/>
+<grid distance="0.05" unitdist="inch" unit="inch" style="lines" multiple="1" display="yes" altdistance="0.025" altunitdist="inch" altunit="inch"/>
 <layers>
 <layer number="1" name="Top" color="4" fill="1" visible="no" active="no"/>
@@
 <part name="IC3" library="we-chip" deviceset="A3909" device="-LY"/>
 <part name="IC4" library="we-chip" deviceset="A3909" device="-LY"/>
-<part name="D2" library="we-rcl" deviceset="D_SCHOTTKY" device="-SMA" value="2A/16V"/>
+<part name="D2" library="we-rcl" deviceset="D_SCHOTTKY" device="-SMA" value="2A/20V"/>
 <part name="GND" library="we-rcl" deviceset="PAD" device="-1.0_NC" value="PAD-1.0_NC"/>
 <part name="GND34" library="supply1" deviceset="GND" device=""/>
@@
 <part name="C13" library="we-rcl" deviceset="CAPACITOR" device="-0402" value="100n"/>
 <part name="GND58" library="supply1" deviceset="GND" device=""/>
-<part name="D6" library="we-rcl" deviceset="D_SCHOTTKY" device="-SMA" value="2A/16V"/>
+<part name="D6" library="we-rcl" deviceset="D_SCHOTTKY" device="-SMA" value="2A/20V"/>
 <part name="C12" library="we-rcl" deviceset="CAPACITOR" device="-0805" value="22u/6.3V"/>
 <part name="R2" library="we-rcl" deviceset="RESISTOR" device="-0402" value="47k"/>
@@
 <part name="R14" library="we-rcl" deviceset="RESISTOR" device="-0402" value="1k"/>
 <part name="R45" library="we-rcl" deviceset="RESISTOR" device="-0402" value="330"/>
-<part name="D5" library="we-rcl" deviceset="D_SCHOTTKY" device="-SMA" value="2A/16V"/>
-<part name="D1" library="we-rcl" deviceset="D_SCHOTTKY" device="-SMA" value="2A/16V"/>
+<part name="D5" library="we-rcl" deviceset="D_SCHOTTKY" device="-SMA" value="2A/20V"/>
+<part name="D1" library="we-rcl" deviceset="D_SCHOTTKY" device="-SMA" value="2A/20V"/>
 <part name="LOGO2" library="we-symbol" deviceset="OSHW_LOGO" device="X0150" value="OSHW_LOGOX0150"/>
 <part name="LOGO4" library="we-symbol" deviceset="LOGO" device="-PLACE"/>
+<part name="FRAME2" library="we-symbol" deviceset="FRAME-A4L" device=""/>
 </parts>
 <sheets>
@@
 </nets>
 </sheet>
+<sheet>
+<plain>
+<wire x1="78.74" y1="170.18" x2="78.74" y2="35.56" width="0.6096" layer="94"/>
+<wire x1="78.74" y1="35.56" x2="137.16" y2="35.56" width="0.6096" layer="94"/>
+<wire x1="137.16" y1="35.56" x2="137.16" y2="170.18" width="0.6096" layer="94"/>
+<wire x1="137.16" y1="170.18" x2="78.74" y2="170.18" width="0.6096" layer="94"/>
+<text x="106.68" y="121.92" size="2.54" layer="94" align="center">SAMD21 + WINC1500</text>
+<text x="106.68" y="132.08" size="3.81" layer="94" align="center">SAMW25 Module</text>
+<text x="40.64" y="81.28" size="3.81" layer="94" rot="R180" align="center">USB</text>
+<wire x1="58.42" y1="88.9" x2="22.86" y2="88.9" width="0.6096" layer="94"/>
+<wire x1="22.86" y1="88.9" x2="22.86" y2="73.66" width="0.6096" layer="94"/>
+<wire x1="22.86" y1="73.66" x2="58.42" y2="73.66" width="0.6096" layer="94"/>
+<wire x1="58.42" y1="73.66" x2="58.42" y2="88.9" width="0.6096" layer="94"/>
+<text x="106.68" y="86.36" size="3.81" layer="94" rot="R180" align="center">ARM Cortex-M0+
+with
+USB + WiFi/WLAN</text>
+<wire x1="157.48" y1="55.88" x2="157.48" y2="35.56" width="0.6096" layer="94"/>
+<wire x1="157.48" y1="35.56" x2="193.04" y2="35.56" width="0.6096" layer="94"/>
+<wire x1="193.04" y1="35.56" x2="193.04" y2="55.88" width="0.6096" layer="94"/>
+<wire x1="193.04" y1="55.88" x2="157.48" y2="55.88" width="0.6096" layer="94"/>
+<wire x1="203.2" y1="170.18" x2="203.2" y2="149.86" width="0.6096" layer="94"/>
+<wire x1="203.2" y1="149.86" x2="238.76" y2="149.86" width="0.6096" layer="94"/>
+<wire x1="238.76" y1="149.86" x2="238.76" y2="170.18" width="0.6096" layer="94"/>
+<wire x1="238.76" y1="170.18" x2="203.2" y2="170.18" width="0.6096" layer="94"/>
+<wire x1="203.2" y1="147.32" x2="203.2" y2="127" width="0.6096" layer="94"/>
+<wire x1="203.2" y1="127" x2="238.76" y2="127" width="0.6096" layer="94"/>
+<wire x1="238.76" y1="127" x2="238.76" y2="147.32" width="0.6096" layer="94"/>
+<wire x1="238.76" y1="147.32" x2="203.2" y2="147.32" width="0.6096" layer="94"/>
+<wire x1="203.2" y1="124.46" x2="203.2" y2="104.14" width="0.6096" layer="94"/>
+<wire x1="203.2" y1="104.14" x2="238.76" y2="104.14" width="0.6096" layer="94"/>
+<wire x1="238.76" y1="104.14" x2="238.76" y2="124.46" width="0.6096" layer="94"/>
+<wire x1="238.76" y1="124.46" x2="203.2" y2="124.46" width="0.6096" layer="94"/>
+<wire x1="203.2" y1="101.6" x2="203.2" y2="81.28" width="0.6096" layer="94"/>
+<wire x1="203.2" y1="81.28" x2="238.76" y2="81.28" width="0.6096" layer="94"/>
+<wire x1="238.76" y1="81.28" x2="238.76" y2="101.6" width="0.6096" layer="94"/>
+<wire x1="238.76" y1="101.6" x2="203.2" y2="101.6" width="0.6096" layer="94"/>
+<wire x1="203.2" y1="55.88" x2="203.2" y2="35.56" width="0.6096" layer="94"/>
+<wire x1="203.2" y1="35.56" x2="238.76" y2="35.56" width="0.6096" layer="94"/>
+<wire x1="238.76" y1="35.56" x2="238.76" y2="55.88" width="0.6096" layer="94"/>
+<wire x1="238.76" y1="55.88" x2="203.2" y2="55.88" width="0.6096" layer="94"/>
+<text x="175.26" y="45.72" size="3.81" layer="94" align="center">2x A3909</text>
+<text x="175.26" y="38.1" size="2.54" layer="94" align="center">Motor Driver</text>
+<text x="220.98" y="162.56" size="3.81" layer="94" align="center">7x
+IOs</text>
+<text x="220.98" y="139.7" size="3.81" layer="94" align="center">2x
+I2C</text>
+<text x="220.98" y="116.84" size="3.81" layer="94" align="center">1x
+UART</text>
+<text x="220.98" y="93.98" size="3.81" layer="94" align="center">1x
+SPI</text>
+<text x="220.98" y="48.26" size="3.81" layer="94" align="center">4x
+Full Bridges</text>
+<wire x1="203.2" y1="78.74" x2="203.2" y2="58.42" width="0.6096" layer="94"/>
+<wire x1="203.2" y1="58.42" x2="238.76" y2="58.42" width="0.6096" layer="94"/>
+<wire x1="238.76" y1="58.42" x2="238.76" y2="78.74" width="0.6096" layer="94"/>
+<wire x1="238.76" y1="78.74" x2="203.2" y2="78.74" width="0.6096" layer="94"/>
+<text x="220.98" y="71.12" size="3.81" layer="94" align="center">1x
+Power Switch</text>
+<wire x1="157.48" y1="78.74" x2="157.48" y2="58.42" width="0.6096" layer="94"/>
+<wire x1="157.48" y1="58.42" x2="193.04" y2="58.42" width="0.6096" layer="94"/>
+<wire x1="193.04" y1="58.42" x2="193.04" y2="78.74" width="0.6096" layer="94"/>
+<wire x1="193.04" y1="78.74" x2="157.48" y2="78.74" width="0.6096" layer="94"/>
+<text x="175.26" y="68.58" size="3.81" layer="94" align="center">1x MosFet</text>
+<text x="40.64" y="55.88" size="3.81" layer="94" rot="R180" align="center">Power Supply</text>
+<wire x1="22.86" y1="63.5" x2="22.86" y2="35.56" width="0.6096" layer="94"/>
+<wire x1="22.86" y1="35.56" x2="58.42" y2="35.56" width="0.6096" layer="94"/>
+<wire x1="58.42" y1="35.56" x2="58.42" y2="63.5" width="0.6096" layer="94"/>
+<wire x1="58.42" y1="63.5" x2="22.86" y2="63.5" width="0.6096" layer="94"/>
+<text x="40.64" y="45.72" size="2.54" layer="94" rot="R180" align="center">7-14V Ext. Power
+or
+5V USB</text>
+<wire x1="203.2" y1="68.58" x2="193.04" y2="68.58" width="0.6096" layer="97"/>
+<wire x1="193.04" y1="45.72" x2="203.2" y2="45.72" width="0.6096" layer="97"/>
+<wire x1="203.2" y1="91.44" x2="137.16" y2="91.44" width="0.6096" layer="97"/>
+<wire x1="203.2" y1="114.3" x2="137.16" y2="114.3" width="0.6096" layer="97"/>
+<wire x1="203.2" y1="137.16" x2="137.16" y2="137.16" width="0.6096" layer="97"/>
+<wire x1="203.2" y1="160.02" x2="137.16" y2="160.02" width="0.6096" layer="97"/>
+<wire x1="58.42" y1="81.28" x2="78.74" y2="81.28" width="0.6096" layer="97"/>
+<wire x1="157.48" y1="68.58" x2="137.16" y2="68.58" width="0.6096" layer="97"/>
+<wire x1="157.48" y1="45.72" x2="137.16" y2="45.72" width="0.6096" layer="97"/>
+<text x="220.98" y="152.4" size="2.54" layer="94" align="center">5V tolerant</text>
+<text x="220.98" y="129.54" size="2.54" layer="94" align="center">5V tolerant</text>
+<text x="220.98" y="106.68" size="2.54" layer="94" align="center">5V tolerant</text>
+<text x="220.98" y="83.82" size="2.54" layer="94" align="center">5V tolerant</text>
+<text x="220.98" y="60.96" size="2.54" layer="94" align="center">up to 2A</text>
+<text x="220.98" y="38.1" size="2.54" layer="94" align="center">up to 1A/phase</text>
+<wire x1="40.64" y1="73.66" x2="40.64" y2="63.5" width="0.6096" layer="97"/>
+<wire x1="40.64" y1="35.56" x2="40.64" y2="30.48" width="0.6096" layer="97"/>
+<wire x1="40.64" y1="30.48" x2="106.68" y2="30.48" width="0.6096" layer="97"/>
+<wire x1="106.68" y1="30.48" x2="175.26" y2="30.48" width="0.6096" layer="97"/>
+<wire x1="175.26" y1="30.48" x2="175.26" y2="35.56" width="0.6096" layer="97"/>
+<text x="162.56" y="22.86" size="1.27" layer="95" align="top-left">Released under the Creative Commons Attribution Share-Alike
+License. http://creativecommons.org/licenses/by-sa/4.0/
+Designed by Watterott electronic (www.watterott.com)</text>
+<wire x1="175.26" y1="30.48" x2="220.98" y2="30.48" width="0.6096" layer="97"/>
+<wire x1="220.98" y1="30.48" x2="220.98" y2="35.56" width="0.6096" layer="97"/>
+<wire x1="220.98" y1="55.88" x2="220.98" y2="58.42" width="0.6096" layer="97"/>
+<wire x1="220.98" y1="78.74" x2="220.98" y2="81.28" width="0.6096" layer="97"/>
+<wire x1="220.98" y1="101.6" x2="220.98" y2="104.14" width="0.6096" layer="97"/>
+<wire x1="220.98" y1="124.46" x2="220.98" y2="127" width="0.6096" layer="97"/>
+<wire x1="220.98" y1="147.32" x2="220.98" y2="149.86" width="0.6096" layer="97"/>
+<wire x1="106.68" y1="30.48" x2="106.68" y2="35.56" width="0.6096" layer="97"/>
+</plain>
+<instances>
+<instance part="FRAME2" gate="F" x="0" y="0"/>
+</instances>
+<busses>
+</busses>
+<nets>
+</nets>
+</sheet>
